Commit message: eliminación de archivos demás para correr la simulación

File: ros2_ws/src/mi_primer_paquete/urdf/robot.urdf (robot description, URDF)
Before this commit: robot mi_robot, 4 links, 3 joints
Links:
- added link world
- link antebrazo_link: geometry visual mesh filename=package://mi_primer_paquete/urdf/Modelos_en_stl/Ensamblaje_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 scale=0.001 0.001 0.001
- link base_link: geometry visual mesh filename=package://mi_primer_paquete/urdf/Modelos_en_stl/Ensamblaje_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 scale=0.001 0.001 0.001
- link brazo_link: geometry visual mesh filename=package://mi_primer_paquete/urdf/Modelos_en_stl/Ensamblaje_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 scale=0.001 0.001 0.001
- link hombro_link: geometry visual mesh filename=package://mi_primer_paquete/urdf/Modelos_en_stl/Ensamblaje_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 scale=0.001 0.001 0.001
Joints:
- added joint world_to_base: type fixed, parent world, child base_link, origin xyz=0 0 0 rpy=0 0 0
- joint joint_brazo_antebrazo: origin xyz=0 0 120 rpy=0 0 0 -> xyz=0 0 0.120 rpy=0 0 0
- joint joint_hombro_brazo: origin xyz=0 0 111.7 rpy=0 0 0 -> xyz=0 0 0.1117 rpy=0 0 0
